File: uswc.kicad_pcb (KiCad board)
At the start: 2 copper layers, 38.8 x 33.3 mm, 65 parts, among them J1 USB_C_Receptacle, J2 debug-port, J3 USB3150-30-130-A, J4 jlink, P1 DFP, SW1 SW_SPDT, SW3 SW_SPDT, SW4 SW_Push, U10 SRV05-4, U2 W25Q32JVZP, U3 74LVC1G3157, U4 RP2040, U5 XC6206PxxxMR, U6 TXB0104RUT, U7 LM397, U9 SRV05-4, Y1 12MHz 10ppm, Y2 12MHz 10ppm

Commit message: 0.2
Parts:
- removed C18: 1uF, Capacitor_SMD:C_0603_1608Metric
- removed J4: jlink, Connector_PinHeader_1.27mm:PinHeader_2x05_P1.27mm_Vertical_SMD
- removed SW3: SW_SPDT, Button_Switch_SMD:SW_SPDT_PCM12
- removed SW4: SW_Push, Button_Switch_SMD:SW_SPST_B3U-1000P
- removed TP10, TP11, TP3, TP4, TP8, TP9: inline, TestPoint:TestPoint_Pad_D1.0mm
- removed TP5: VBUS, TestPoint:TestPoint_THTPad_D1.5mm_Drill0.7mm
- removed TP6: GND, TestPoint:TestPoint_Bridge_Pitch2.0mm_Drill0.7mm
- removed TP7: 3V3, TestPoint:TestPoint_THTPad_D1.5mm_Drill0.7mm
- removed U17: ~, Package_DFN_QFN:UQFN-16_1.8x2.6mm_P0.4mm
- added C2: 1uF, Capacitor_SMD:C_0603_1608Metric, F.Cu at (76.0, 125.0)
- added R11: 5.1k, Resistor_SMD:R_0603_1608Metric, F.Cu at (89.1, 111.3)
- added R12: 56k, Resistor_SMD:R_0603_1608Metric, F.Cu at (92.1, 111.3)
- added R13: 56k, Resistor_SMD:R_0603_1608Metric, F.Cu at (89.1, 112.8)
- added R5: 56k, Resistor_SMD:R_0603_1608Metric, F.Cu at (73.7, 124.3)
- added R6: 56k, Resistor_SMD:R_0603_1608Metric, F.Cu at (78.3, 128.8)
- added R7: 56k, Resistor_SMD:R_0603_1608Metric, F.Cu at (76.0, 128.0)
- added REF**: header-bites, uswc:header-bites, F.Cu at (81.6, 119.0)
- added U13: LM2903, Package_DFN_QFN:DFN-8-1EP_2x2mm_P0.5mm_EP0.9x1.6mm, F.Cu at (85.5, 115.9)
- added U8: TS5A23166DCU, Package_SO:VSSOP-8_2.3x2mm_P0.5mm, F.Cu at (85.7, 111.9)
- J1: footprint Connector_USB:USB_C_Receptacle_Amphenol_12401548E4-2A -> Connector_USB:USB_C_Receptacle_Molex_105450-0101
- J2: value debug-port -> Conn_01x02_Socket; footprint misc:debug-port-single-side -> Connector_PinHeader_2.00mm:PinHeader_1x02_P2.00mm_Vertical
- J3: value USB3150-30-130-A -> Conn_01x08_Pin; footprint lib:USB3150-30-130-A -> Connector_PinHeader_2.54mm:PinHeader_1x08_P2.54mm_Vertical
- TP1: value inline -> SWC_L; moved to B.Cu
- TP2: value inline -> SWD_L; moved to B.Cu
- U3: value 74LVC1G3157 -> SN74LVC1T45DBV; footprint Package_TO_SOT_SMD:SOT-363_SC-70-6 -> Package_TO_SOT_SMD:SOT-23-6
- U6: value TXB0104RUT -> 74LVC1G125; footprint Package_DFN_QFN:Texas_R-PUQFN-N12 -> Package_TO_SOT_SMD:SOT-23-5
- moved R16 26.1 mm to (92.1, 112.8), turned to 0 degrees
- moved R10 16.9 mm to (60.2, 126.2), turned to -90 degrees
- moved C19 16.7 mm to (78.3, 127.3), turned to 180 degrees
- moved U5 16.6 mm to (78.5, 124.5), turned to 90 degrees
- moved R23 14.9 mm to (70.4, 132.2)
- moved SW1 14.9 mm to (75.6, 132.0)
- moved R2 14.0 mm to (86.0, 126.1), turned to 180 degrees
- moved U11 11.0 mm to (63.5, 127.6), turned to -90 degrees
- moved U7 9.84 mm to (73.2, 126.8), turned to 180 degrees
- moved C14 8.13 mm to (86.8, 122.3), turned to -90 degrees
- moved J2 7.61 mm to (80.9, 107.2), turned to 180 degrees
- moved U14 7.58 mm to (63.5, 123.3), turned to 180 degrees
- moved TP1 7.55 mm to (62.7, 125.3), turned to 180 degrees
- moved U9 6.76 mm to (85.5, 119.0), turned to 180 degrees
- moved TP2 6.61 mm to (65.6, 122.8), turned to 180 degrees
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Connections:
- net Net-(J1-CC1) renamed CC1
- net Net-(J1-CC2) renamed CC2
- J1 pad A8: unconnected-(J1-SBU1-PadA8) -> +3V3
- J1 pad B2: unconnected-(J1-TX2+-PadB2) -> DBG_SWC_S
- J1 pad B3: unconnected-(J1-TX2--PadB3) -> DBG_SWD_S
- J2 pad 2: +3V3 -> BOOT
- J3 pad 1: VBUS -> SHIELD
- J3 pad 2: JLK_D- -> GND
- J3 pad 3: JLK_D+ -> VBUS
- J3 pad 4: unconnected-(J3-ID-Pad4) -> D-
- J3 pad 5: GND -> D+
- J3 pad 6: SHIELD -> DBG_SWC
- P1 pad A10: SS_A10 -> SS_X-
- P1 pad A11: SS_A11 -> SS_X+
- P1 pad A2: unconnected-(P1-TX1+-PadA2) -> SS_X+
- P1 pad A3: unconnected-(P1-TX1--PadA3) -> SS_X-
- P1 pad B10: SS_B10 -> SS_X-
- P1 pad B11: SS_B11 -> SS_X+
- P1 pad B2: unconnected-(P1-TX2+-PadB2) -> SS_X+
- P1 pad B3: unconnected-(P1-TX2--PadB3) -> SS_X-
- R10 pad 1: DUT_VREF -> +3V3
- R10 pad 2: +3V3 -> DUT_SBU_SWD_ALT
- R16 pad 1: SS_DIR -> +3V3
- R16 pad 2: +3V3 -> Net-(R12-Pad1)
- TP1 pad 1: /DUT_SWD/TMS -> DUT_SWC_L
- TP2 pad 1: /DUT_SWC/TCK -> DUT_SWD_L
- U1 pad 1: DAP_D- -> DUT_D-
- U1 pad 2: DAP_D+ -> DUT_D+
- U1 pad 3: DUT_D- -> DAP_D-
- U1 pad 4: DUT_D+ -> DAP_D+
- U1 pad 7: JLK_D- -> unconnected-(U1-DM1--Pad7)
- U1 pad 8: JLK_D+ -> unconnected-(U1-DP1+-Pad8)
- U11 pad 1: DUT_SWD/TMS_J -> DUT_SWD
- U11 pad 11: DUT_TDI_P -> unconnected-(U11-S4B-Pad11)
- U11 pad 12: /DUT_TDI -> unconnected-(U11-D4-Pad12)
- U11 pad 13: DUT_TDI_J -> unconnected-(U11-S4A-Pad13)
- U11 pad 15: DUT_SWD/TMS_P -> DUT_SWC
- U11 pad 16: /DUT_SWD/TMS -> DUT_SWC/D_SBU
- U11 pad 2: USE_PICO -> DUT_SBU_SWD_ALT
- U11 pad 3: DUT_SWC/TCK_P -> DUT_SWD
- U11 pad 4: /DUT_SWC/TCK -> DUT_SWD/C_SBU
- U11 pad 5: DUT_SWC/TCK_J -> DUT_SWC
- U11 pad 7: DUT_SWO/TDO_P -> unconnected-(U11-S3B-Pad7)
- U11 pad 8: /DUT_SWO/TDO -> unconnected-(U11-D3-Pad8)
- U11 pad 9: DUT_SWO/TDO_J -> unconnected-(U11-S3A-Pad9)
- U14 pad 11: DUT_SWD/C_SBU -> DUT_SWC_L
- U14 pad 12: /DUT_SWD/TMS -> SS_X+
- U14 pad 13: DUT_SWC/D_SBU -> unconnected-(U14-S4A-Pad13)
- U14 pad 15: DUT_VREF_B -> DUT_VREF
- U14 pad 3: DUT_VREF_A -> DUT_VREF
- U14 pad 7: DUT_SWC/D_SBU -> DUT_SWD_L
- U14 pad 8: /DUT_SWC/TCK -> SS_X-
- U14 pad 9: DUT_SWD/C_SBU -> unconnected-(U14-S3A-Pad9)
- U3 pad 1: DUT_VREF_A -> DUT_VREF
- U3 pad 3: DUT_VREF_B -> DUT_SWD_L
- U3 pad 4: DUT_VREF -> DUT_SWD
- U3 pad 5: +3V3 -> DUT_SWDIR
- U3 pad 6: SS_DIR -> +3V3
- U4 pad 15: DUT_SWC/TCK_P -> unconnected-(U4-GPIO12-Pad15)
- U4 pad 16: DUT_SWD/TMS_P -> unconnected-(U4-GPIO13-Pad16)
- U4 pad 17: DUT_SWO/TDO_P -> unconnected-(U4-GPIO14-Pad17)
- U4 pad 18: DUT_TDI_P -> unconnected-(U4-GPIO15-Pad18)
- U4 pad 26: unconnected-(U4-RUN-Pad26) -> +3V3
- U4 pad 35: unconnected-(U4-GPIO23-Pad35) -> DUT_SWDIR
- U4 pad 36: unconnected-(U4-GPIO24-Pad36) -> DUT_SWC
- U4 pad 37: unconnected-(U4-GPIO25-Pad37) -> DUT_SWD
- U6 pad 1: DUT_VREF -> GND
- U6 pad 2: /SS_B10_NORM -> DUT_SWC
- U6 pad 3: /SS_B11_NORM -> GND
- U6 pad 4: /SS_A10_NORM -> DUT_SWC_L
- U6 pad 5: /SS_A11_NORM -> DUT_VREF
- U7 pad 1: DUT_VREF_A -> Net-(U7--)
- U7 pad 3: DUT_VREF_B -> Net-(U7-+)
- U7 pad 4: SS_DIR -> DUT_SBU_SWD_ALT
Routing:
- net DUT_SWC: track 0.00 -> 29.8 mm, vias 0 -> 4
- net GND: track 107.4 -> 135.8 mm, vias 41 -> 40
- net SS_X+: track 0.00 -> 27.0 mm, vias 0 -> 5
- net SS_DIR: track 25.2 -> 0.00 mm, vias 5 -> 0
- net +3V3: track 144.9 -> 168.7 mm, vias 11 -> 15
- net SS_X-: track 0.00 -> 22.7 mm, vias 0 -> 4
- net DUT_SWD: track 0.00 -> 22.3 mm, vias 0 -> 2
- net JLK_D+: track 21.2 -> 0.00 mm, vias 1 -> 0
- net DUT_VREF_B: track 20.8 -> 0.00 mm, vias 3 -> 0
- net SS_A11: track 20.8 -> 0.00 mm, vias 3 -> 0
- net JLK_D-: track 20.5 -> 0.00 mm, vias 1 -> 0
- net SS_A10: track 20.5 -> 0.00 mm, vias 2 -> 0
- net DUT_SBU_SWD_ALT: track 0.00 -> 20.0 mm, vias 0 -> 2
- net SS_B10: track 17.1 -> 0.00 mm, vias 3 -> 0
- net DUT_VREF_A: track 14.5 -> 0.00 mm, vias 4 -> 0
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- removed copper zone on F.Cu, net SHIELD
Other:
- board size 38.8 x 33.3 mm -> 43.3 x 30 mm
- board text added: "BOOT"
- board text added: "T2"
