File: uswc.kicad_pcb (KiCad board)
At the start: 2 copper layers, 43.3 x 30 mm, 61 parts, among them J1 USB_C_Receptacle, J2 Conn_01x02_Socket, J3 Conn_01x08_Pin, P1 DFP, SW1 SW_SPDT, U10 SRV05-4, U13 LM2903, U2 W25Q32JVZP, U3 SN74LVC1T45DBV, U4 RP2040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

Commit message: backup
Parts:
- removed C2, C5: 1uF, Capacitor_SMD:C_0603_1608Metric
- removed C7: 0.1uF, Capacitor_SMD:C_0603_1608Metric
- removed J3: Conn_01x08_Pin, Connector_PinHeader_2.54mm:PinHeader_1x08_P2.54mm_Vertical
- removed R10, R12, R13, R16, R5, R6, R7: 56k, Resistor_SMD:R_0603_1608Metric
- removed R11, R22, R23: 5.1k, Resistor_SMD:R_0603_1608Metric
- removed REF**: header-bites, uswc:header-bites
- removed U1: ~, Package_SO:QSOP-16_3.9x4.9mm_P0.635mm
- removed U13: LM2903, Package_DFN_QFN:DFN-8-1EP_2x2mm_P0.5mm_EP0.9x1.6mm
- removed U8: TS5A23166DCU, Package_SO:VSSOP-8_2.3x2mm_P0.5mm
- removed Y1: 12MHz 10ppm, Crystal:Crystal_SMD_3225-4Pin_3.2x2.5mm
- J1: value USB_C_Receptacle -> USB_C_Receptacle_USB2.0_16P; footprint Connector_USB:USB_C_Receptacle_Molex_105450-0101 -> Connector_USB:USB_C_Receptacle_HRO_TYPE-C-31-M-12
- U7: value LM397 -> CH334F; footprint Package_TO_SOT_SMD:SOT-23-5 -> Package_DFN_QFN:QFN-24-1EP_4x4mm_P0.5mm_EP2.7x2.7mm
- moved R1 17.1 mm to (77.4, 109.8)
- moved R2 17.1 mm to (77.4, 111.3)
- moved C14 14.1 mm to (74.5, 115.4)
- moved U9 12.5 mm to (73.2, 121.1), turned to 0 degrees
- moved J1 11.7 mm to (80.6, 117.4)
- moved C1 8.93 mm to (67.3, 117.2), turned to 0 degrees
- moved SW1 7.94 mm to (79.7, 125.2)
- moved U7 7.79 mm to (68.5, 120.6), turned to 0 degrees
- moved C20 7.74 mm to (74.5, 112.4)
- moved R14 7.68 mm to (73.0, 112.4), turned to 90 degrees
- moved R9 6.89 mm to (59.5, 116.4), turned to 0 degrees
- moved U5 5.29 mm to (73.4, 125.9)
- moved C3 5.22 mm to (70.7, 113.3), turned to -90 degrees
- moved C19 5.09 mm to (73.4, 128.7)
- moved J2 4.30 mm to (76.6, 107.2)
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Connections:
- C1 pad 2: Net-(U1-VDD33) -> Net-(U7-VDD33)
- J1 pad A8: +3V3 -> DBG_SWD
- J1 pad B8: unconnected-(J1-SBU2-PadB8) -> DBG_SWC
- P1 pad A5: Net-(P1-CC) -> DFP_CC1
- P1 pad B5: Net-(P1-VCONN) -> DFP_CC2
- R8 pad 1: Net-(P1-CC) -> DFP_CC1
- R9 pad 1: Net-(P1-VCONN) -> DFP_CC2
- SW1 pad 1: Net-(SW1-A) -> GND
- SW1 pad 3: Net-(SW1-C) -> +3V3
- U3 pad 1: DUT_VREF -> +3V3
- U3 pad 3: DUT_SWD_L -> DUT_SWD
- U3 pad 4: DUT_SWD -> DUT_SWD_L
- U3 pad 6: +3V3 -> DUT_VREF
- U4 pad 34: unconnected-(U4-GPIO22-Pad34) -> DUT_SBU_SWD_ALT
- U4 pad 38: unconnected-(U4-GPIO26_ADC0-Pad38) -> DFP_CC1
- U4 pad 39: unconnected-(U4-GPIO27_ADC1-Pad39) -> DFP_CC2
- U4 pad 40: unconnected-(U4-GPIO28_ADC2-Pad40) -> DUT_SWD/C_SBU
- U4 pad 41: unconnected-(U4-GPIO29_ADC3-Pad41) -> DUT_SWC/D_SBU
- U7 pad 1: Net-(U7--) -> unconnected-(U7-~{OVCUR}-Pad1)
- U7 pad 2: GND -> unconnected-(U7-NC-Pad2)
- U7 pad 3: Net-(U7-+) -> unconnected-(U7-XO-Pad3)
- U7 pad 4: DUT_SBU_SWD_ALT -> GND
- U7 pad 5: +3V3 -> DUT_D-
Routing:
- net +3V3: track 168.7 -> 103.6 mm, vias 15 -> 10
- net GND: track 135.8 -> 86.7 mm, vias 40 -> 37
- net DUT_SBU_SWD_ALT: track 20.0 -> 0.00 mm, vias 2 -> 0
- net VBUS: track 85.9 -> 71.4 mm, vias 7 -> 11
- net Net-(U13A--): track 14.4 -> 0.00 mm, vias 3 -> 0
- net Net-(U8-IN1): track 13.1 -> 0.00 mm, vias 2 -> 0
- net CC2: track 18.7 -> 6.22 mm, vias 3 -> 0
- net D+: track 22.7 -> 10.2 mm, vias 2 -> 0
- net USE_SS: track 17.2 -> 4.95 mm, vias 2 -> 1
- net DBG_SWD_S: track 11.3 -> 0.00 mm, vias 2 -> 0
- net DBG_SWC_S: track 10.5 -> 0.00 mm, vias 2 -> 0
- net DUT_SWD/C_SBU: track 17.1 -> 7.84 mm
- net Net-(U1-XO): track 8.19 -> 0.00 mm
- net SHIELD: track 42.0 -> 50.1 mm
- net D-: track 19.5 -> 12.8 mm, vias 1 -> 0
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Other:
- board size 43.3 x 30 mm -> 31 x 26.8 mm
- board text added: "SB"
- board text added: "v0.3"
- board text removed: "SS"
- board text removed: "T2"
- board text removed: "v0.2"

Commit message: pend
Parts:
- removed SW1: SW_SPDT, Button_Switch_SMD:SW_SPDT_PCM12
- removed U11, U14: ~, Package_DFN_QFN:UQFN-16_1.8x2.6mm_P0.4mm
- added C2: 1u, Capacitor_SMD:C_0603_1608Metric, F.Cu at (67.6, 129.4)
- added R5: 56k, Resistor_SMD:R_0603_1608Metric, F.Cu at (62.6, 121.4)
- added R6: 56k, Resistor_SMD:R_0603_1608Metric, F.Cu at (58.5, 127.8)
- added R7: 5.1k, Resistor_SMD:R_0603_1608Metric, F.Cu at (68.4, 125.5)
- added U1: ADG884xRM, Package_SO:MSOP-10_3x3mm_P0.5mm, F.Cu at (62.6, 125.1)
- added U8: ADG884xRM, Package_SO:MSOP-10_3x3mm_P0.5mm, F.Cu at (62.6, 128.6)
- P1: footprint lib:jingtuojin_918-118A2021Y40005 -> lib:jingtuojin_918-118A2021Y40005-no-ss
- TP1, TP2: moved to F.Cu
- moved R9 5.25 mm to (61.1, 121.4), turned to -90 degrees
- moved TP1 4.94 mm to (67.1, 127.6), turned to 0 degrees
- moved C14 4.68 mm to (71.0, 118.5), turned to 180 degrees
- moved U5 4.50 mm to (77.9, 125.8), turned to 180 degrees
- moved R14 4.16 mm to (76.6, 110.3), turned to -90 degrees
- moved C19 3.34 mm to (75.1, 125.8), turned to -90 degrees
- moved U10 2.35 mm to (60.8, 117.5)
- moved C15 2.26 mm to (56.2, 124.7)
- moved U3 2.10 mm to (71.2, 125.3)
- moved U6 2.10 mm to (71.2, 128.7)
- moved FB1 2.00 mm to (55.6, 122.7)
- moved TP2 1.85 mm to (66.7, 124.3), turned to 0 degrees
- moved R8 1.80 mm to (59.6, 121.4)
- moved C1 1.80 mm to (65.5, 117.2)
- moved C20 1.70 mm to (72.8, 112.3)
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Connections:
- U4 pad 30: unconnected-(U4-GPIO19-Pad30) -> DUT_SWD_CONN
- U4 pad 31: unconnected-(U4-GPIO20-Pad31) -> DUT_SWD_SWAP
- U4 pad 32: unconnected-(U4-GPIO21-Pad32) -> PWM
- U4 pad 34: DUT_SBU_SWD_ALT -> unconnected-(U4-GPIO22-Pad34)
- U4 pad 39: DFP_CC2 -> DUT_SBU_B
- U4 pad 40: DUT_SWD/C_SBU -> DFP_CC2
- U4 pad 41: DUT_SWC/D_SBU -> DUT_SBU_A
Routing:
- net SS_X+: track 26.9 -> 0.00 mm, vias 5 -> 0
- net GND: track 86.7 -> 112.5 mm
- net DUT_SWD_SWAP: track 0.00 -> 25.5 mm, vias 0 -> 3
- net SS_X-: track 24.7 -> 0.00 mm, vias 4 -> 0
- net DUT_SBU_A: track 12.8 -> 34.2 mm, vias 2 -> 4
- net DFP_CC2: track 0.90 -> 20.6 mm, vias 0 -> 2
- net DUT_SBU_B: track 10.8 -> 29.1 mm, vias 1 -> 2
- net DUT_SWD_CONN: track 0.00 -> 16.0 mm, vias 0 -> 2
- net DFP_CC1: track 3.21 -> 18.6 mm, vias 0 -> 2
- net PWM: track 0.00 -> 14.0 mm, vias 0 -> 2
- net DUT_SWC: track 29.4 -> 20.3 mm, vias 4 -> 2
- net DUT_SWD_L: track 7.15 -> 16.2 mm
- net DUT_SWD: track 22.6 -> 14.0 mm
- net DUT_VREF: track 13.6 -> 6.57 mm, vias 2 -> 0
- net +3V3: track 103.6 -> 98.4 mm, vias 10 -> 8
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Other:
- board size 31 x 26.8 mm -> 29.3 x 26.8 mm
- board text removed: "SB"
- board text removed: "SBU"

Commit message: v0.3
Parts:
- added TP3: -, TestPoint:TestPoint_Pad_D1.0mm, B.Cu at (61.0, 104.8)
- added TP4: +, TestPoint:TestPoint_Pad_D1.0mm, B.Cu at (59.4, 104.8)
- added TP5: +, TestPoint:TestPoint_Pad_D1.0mm, B.Cu at (57.9, 105.2)
- C2: value 1u -> 10u
- R7: value 5.1k -> 1k
- moved U1 0.40 mm to (62.6, 125.5)
- moved U8 0.40 mm to (62.6, 129.0)
- moved R15 0.30 mm to (60.0, 114.5)
Connections:
- P1 pad B6: (no net) -> AUX_D+
- P1 pad B7: (no net) -> AUX_D-
- U10 pad 4: DUT_D- -> AUX_D+
- U10 pad 6: DUT_D+ -> AUX_D-
- U4 pad 14: unconnected-(U4-GPIO11-Pad14) -> Net-(U4-GPIO11)
- U4 pad 15: unconnected-(U4-GPIO12-Pad15) -> Net-(U4-GPIO12)
- U4 pad 16: unconnected-(U4-GPIO13-Pad16) -> Net-(U4-GPIO13)
- U7 pad 1: unconnected-(U7-~{OVCUR}-Pad1) -> VBUS
Routing:
- net VBUS: track 69.5 -> 75.3 mm, vias 11 -> 14
- net Net-(U4-GPIO13): track 0.00 -> 5.61 mm, vias 0 -> 1
- net Net-(U4-GPIO12): track 0.00 -> 4.19 mm, vias 0 -> 1
- net unconnected-(U7-DP3+-Pad8): track 0.00 -> 3.36 mm
- net AUX_D+: track 0.00 -> 3.34 mm, vias 0 -> 1
- net AUX_D-: track 0.00 -> 3.24 mm, vias 0 -> 1
- net Net-(U4-GPIO11): track 0.00 -> 3.17 mm, vias 0 -> 1
- net unconnected-(U7-DM3--Pad7): track 0.00 -> 2.00 mm
- net DUT_D+: track 10.4 -> 11.6 mm
- net GND: track 112.5 -> 113.3 mm
- net DUT_SWC_L: track 12.7 -> 13.5 mm
- net +3V3: track 98.4 -> 99.0 mm
- net DUT_SBU_A: track 34.2 -> 34.7 mm
- net DUT_SBU_B: track 29.1 -> 29.6 mm

Commit message: v0.4
Parts:
- added C5: 0.1u, Capacitor_SMD:C_0603_1608Metric, F.Cu at (62.1, 127.2)
- added R10: 118k, Resistor_SMD:R_0603_1608Metric, F.Cu at (73.2, 126.5)
- C2: value 10u -> 0.1u
- R5: value 56k -> 10k
- R6: value 56k -> 64.9k
- R8, R9: value 56k -> 36k
- TP1: value SWC_L -> SBU_D
- TP2: value SWD_L -> SBU_C
- U1: value ADG884xRM -> LMV321; footprint Package_SO:MSOP-10_3x3mm_P0.5mm -> Package_TO_SOT_SMD:SOT-353_SC-70-5
- U2: footprint Package_SON:WSON-8-1EP_6x5mm_P1.27mm_EP3.4x4.3mm -> Package_SON:Winbond_USON-8-1EP_3x2mm_P0.5mm_EP0.2x1.6mm
- U3: footprint Package_TO_SOT_SMD:SOT-23-6 -> Package_TO_SOT_SMD:SOT-363_SC-70-6
- U6: value 74LVC1G125 -> SN74LVC1T45DBV; footprint Package_TO_SOT_SMD:SOT-23-5 -> Package_TO_SOT_SMD:SOT-363_SC-70-6
- U8: value ADG884xRM -> MCP1824; footprint Package_SO:MSOP-10_3x3mm_P0.5mm -> Package_TO_SOT_SMD:TSOT-23-5
- Y2: footprint Crystal:Crystal_SMD_3225-4Pin_3.2x2.5mm -> Crystal:Crystal_SMD_2016-4Pin_2.0x1.6mm
- moved U6 12.1 mm to (61.5, 121.4), turned to -90 degrees
- moved U3 9.44 mm to (61.8, 124.4)
- moved TP1 8.56 mm to (59.2, 124.3)
- moved U1 8.45 mm to (71.0, 126.4), turned to 90 degrees
- moved C2 8.13 mm to (73.5, 123.8), turned to 0 degrees
- moved TP2 7.74 mm to (59.2, 122.4)
- moved R6 6.06 mm to (64.4, 126.4), turned to 90 degrees
- moved U8 5.59 mm to (67.5, 126.3), turned to 180 degrees
- moved R15 5.20 mm to (57.4, 110.0), turned to -90 degrees
- moved C17 4.32 mm to (57.4, 107.0), turned to 90 degrees
- moved R5 3.47 mm to (64.9, 124.0), turned to 0 degrees
- moved C19 3.10 mm to (75.9, 122.8), turned to 90 degrees
- moved R2 3.07 mm to (77.9, 108.4)
- moved U5 2.87 mm to (78.7, 123.0), turned to 0 degrees
- moved C15 2.72 mm to (55.9, 122.0)
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Connections:
- C2 pad 1: DUT_VREF -> Net-(U1-+)
- P1 pad A8: DUT_SBU_A -> SBU_D
- P1 pad B6: AUX_D+ -> unconnected-(P1-D+-PadB6)
- P1 pad B7: AUX_D- -> unconnected-(P1-D--PadB7)
- P1 pad B8: DUT_SBU_B -> SBU_C
- R5 pad 1: GND -> Net-(U8-SENSE/ADJ)
- R5 pad 2: DUT_SWD_CONN -> GND
- R6 pad 1: GND -> DUT_VREF
- R6 pad 2: DUT_SWD_SWAP -> Net-(U8-SENSE/ADJ)
- R7 pad 1: DUT_VREF -> Net-(U1-+)
- R8 pad 2: VBUS -> +3V3
- R9 pad 2: VBUS -> +3V3
- TP1 pad 1: DUT_SWC_L -> SBU_D
- TP2 pad 1: DUT_SWD_L -> SBU_C
- U1 pad 1: +3V3 -> Net-(U1-+)
- U1 pad 2: DUT_SWC/D_SBU -> GND
- U1 pad 3: DUT_SBU_B -> MARGIN
- U1 pad 4: DUT_SWD_CONN -> MARGIN
- U1 pad 5: unconnected-(U1-S1B-Pad5) -> +3V3
- U10 pad 4: AUX_D+ -> DUT_D-
- U10 pad 6: AUX_D- -> DUT_D+
- U3 pad 4: DUT_SWD_L -> SBU_D
- U3 pad 5: DUT_SWDIR -> DUT_SWDIR_D
- U4 pad 30: DUT_SWD_CONN -> unconnected-(U4-GPIO19-Pad30)
- U4 pad 31: DUT_SWD_SWAP -> unconnected-(U4-GPIO20-Pad31)
- U4 pad 32: PWM -> DUT_SWDIR_D
- U4 pad 34: unconnected-(U4-GPIO22-Pad34) -> DUT_SWC
- U4 pad 35: DUT_SWDIR -> DUT_SWDIR_C
- U4 pad 36: DUT_SWC -> DUT_SWD
- U4 pad 37: DUT_SWD -> PWM
- U4 pad 39: DUT_SBU_B -> SBU_C
- U4 pad 41: DUT_SBU_A -> SBU_D
- U6 pad 1: GND -> +3V3
- U6 pad 2: DUT_SWC -> GND
- U6 pad 3: GND -> DUT_SWC
- U6 pad 4: DUT_SWC_L -> SBU_C
- U6 pad 5: DUT_VREF -> DUT_SWDIR_C
- U8 pad 2: DUT_SWC_L -> GND
- U8 pad 3: DUT_SWD/C_SBU -> +3V3
- U8 pad 4: DUT_SWD_SWAP -> Net-(U8-SENSE/ADJ)
- U8 pad 5: DUT_SWD_L -> DUT_VREF
Routing:
- net DUT_SBU_A: track 34.7 -> 0.00 mm, vias 4 -> 0
- net SBU_D: track 0.00 -> 32.9 mm, vias 0 -> 4
- net DUT_SBU_B: track 29.6 -> 0.00 mm, vias 2 -> 0
- net DUT_SWD_SWAP: track 26.0 -> 0.00 mm, vias 3 -> 0
- net SBU_C: track 0.00 -> 23.5 mm, vias 0 -> 2
- net DUT_SWDIR_D: track 0.00 -> 17.6 mm, vias 0 -> 2
- net DUT_SWD_L: track 16.6 -> 0.00 mm, vias 2 -> 0
- net DUT_SWD_CONN: track 16.4 -> 0.00 mm, vias 2 -> 0
- net +3V3: track 99.0 -> 114.6 mm, vias 8 -> 11
- net GND: track 113.3 -> 98.2 mm, vias 37 -> 44
- net DUT_SWDIR_C: track 0.00 -> 14.4 mm, vias 0 -> 2
- net DUT_SWDIR: track 14.1 -> 0.00 mm, vias 2 -> 0
- net DUT_SWC_L: track 13.5 -> 0.00 mm, vias 4 -> 0
- net Net-(U8-SENSE/ADJ): track 0.00 -> 11.7 mm, vias 0 -> 2
- net SHIELD: track 54.2 -> 43.6 mm
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Other:
- board size 29.3 x 26.8 mm -> 27.5 x 24 mm
- board text added: "C D"
- board text added: "v0.4"
- board text removed: "JLCJLCJLCJLC"
- board text removed: "v0.3"
