File: uswc.kicad_sch (KiCad schematic)
At the start: 54 parts, among them J1 USB_C_Receptacle, J2 debug-port, J3 USB3150-30-130-A, J4 jlink, P1 DFP, SW1 SW_SPDT, SW3 SW_SPDT, SW4 SW_Push, U10 SRV05-4, U2 W25Q32JVZP, U3 SN74LVC1T45DBV, U4 RP2040, U5 XC6206PxxxMR, U6 74LVC1G125, U9 SRV05-4, Y1 12MHz 10ppm, Y2 12MHz 10ppm

Commit message: 0.2
Parts:
- removed C18: 1uF, Capacitor_SMD:C_0603_1608Metric, symbol Device:C_Small
- removed J2: debug-port, misc:debug-port-single-side, symbol misc:debug-port
- removed J3: USB3150-30-130-A, lib:USB3150-30-130-A, symbol Connector:USB_B_Micro
- removed J4: jlink, Connector_PinHeader_1.27mm:PinHeader_2x05_P1.27mm_Vertical_SMD, symbol misc:jlink
- removed SW3: SW_SPDT, Button_Switch_SMD:SW_SPDT_PCM12, symbol Switch:SW_SPDT
- removed SW4: SW_Push, Button_Switch_SMD:SW_SPST_B3U-1000P, symbol Switch:SW_Push
- removed TP5: VBUS, TestPoint:TestPoint_THTPad_D1.5mm_Drill0.7mm, symbol Connector:TestPoint
- removed TP6: GND, TestPoint:TestPoint_Bridge_Pitch2.0mm_Drill0.7mm, symbol Connector:TestPoint
- removed TP7: 3V3, TestPoint:TestPoint_THTPad_D1.5mm_Drill0.7mm, symbol Connector:TestPoint
- added C2: 1uF, Capacitor_SMD:C_0603_1608Metric, symbol Device:C_Small
- added J2: Conn_01x02_Socket, Connector_PinHeader_2.00mm:PinHeader_1x02_P2.00mm_Vertical, symbol Connector:Conn_01x02_Socket
- added J3: Conn_01x08_Pin, Connector_PinHeader_2.54mm:PinHeader_1x08_P2.54mm_Vertical, symbol Connector:Conn_01x08_Pin
- added R11: 5.1k, Resistor_SMD:R_0603_1608Metric, symbol Device:R
- added R12, R13, R16, R5, R6, R7: 56k, Resistor_SMD:R_0603_1608Metric, symbol Device:R
- added TP1: SWC_L, TestPoint:TestPoint_Pad_D1.0mm, symbol Connector:TestPoint_Small
- added TP2: SWD_L, TestPoint:TestPoint_Pad_D1.0mm, symbol Connector:TestPoint_Small
- added U13: LM2903, Package_DFN_QFN:DFN-8-1EP_2x2mm_P0.5mm_EP0.9x1.6mm, symbol uswc:LM2903DSG
- added U7: LM397, Package_TO_SOT_SMD:SOT-23-5, symbol Comparator:LM397
- added U8: TS5A23166DCU, Package_SO:VSSOP-8_2.3x2mm_P0.5mm, symbol uswc:TS5A23166DCU
- J1: footprint Connector_USB:USB_C_Receptacle_Amphenol_12401548E4-2A -> Connector_USB:USB_C_Receptacle_Molex_105450-0101; LCSC# (none) -> C134092
- U3: LCSC# (none) -> C168856
- U6: footprint (none) -> Package_TO_SOT_SMD:SOT-23-5; LCSC# (none) -> C354448
Connections:
- net DUT_SWC_J is gone; now on net DUT_SWC: U11.5 (S2A)
- net DUT_SWD_J is gone; now on net DUT_SWD: U11.1 (S1A)
- net DUT_VREF_A is gone; now on net DUT_VREF: U14.3 (S2B)
- net DUT_VREF_B is gone; now on net DUT_VREF: U14.15 (S1B)
- net SS_AB10 is gone; now on net SS_X-: P1.A10 (RX2-), P1.B10 (RX1-), U14.8 (D3)
- net SS_AB11 is gone; now on net SS_X+: P1.A11 (RX2+), P1.B11 (RX1+), U14.12 (D4)
- net +3V3: now also J1.A8 (SBU1), R10.1, U4.26 (RUN), J3.8 (Pin_8), R13.1, R16.1, R6.1, U13.8 (V+), U7.5 (V+), U8.8 (VCC); no longer R10.2
- net BOOT: now also J2.2 (Pin_2)
- net D+: now also J3.5 (Pin_5)
- net D-: now also J3.4 (Pin_4)
- net DAP_D+: now also U1.4 (DP3+); no longer U1.2 (DP4+)
- net DAP_D-: now also U1.3 (DM3-); no longer U1.1 (DM4-)
- net DBG_SWC: now also J3.6 (Pin_6), U8.1 (NO1)
- net DBG_SWD: now also J3.7 (Pin_7), U8.5 (NO2)
- net DUT_D+: now also U1.2 (DP4+); no longer U1.4 (DP3+)
- net DUT_D-: now also U1.1 (DM4-); no longer U1.3 (DM3-)
- net DUT_SWC: now also U11.15 (S1B), U4.36 (GPIO24), U6.2; no longer U11.4 (D2), U14.11 (S4B)
- net DUT_SWC/D_SBU: now also U11.16 (D1)
- net DUT_SWD: now also U11.3 (S2B), U3.4 (B), U4.37 (GPIO25); no longer U11.16 (D1), U14.7 (S3B)
- net DUT_SWD/C_SBU: now also U11.4 (D2), R5.2
- net DUT_VREF: no longer R10.1
- net GND: now also C2.2, J2.1 (Pin_1), J3.2 (Pin_2), R11.1, R7.1, U13.4 (V-), U13.9 (V-), U7.2 (V-), U8.4 (GND)
- net SHIELD: now also J3.1 (Pin_1)
- net VBUS: now also J3.3 (Pin_3)
- net CC2: now reaches J1.B5 (CC2), R2.1
- net CC2: now also U13.5 (+)
- net CC1: now reaches J1.A5 (CC1), R1.1
- net CC1: now also U13.3 (+)
- net DUT_SWDIR: now reaches U4.35 (GPIO23)
- net DUT_SWDIR: now also U3.5 (DIR)
- net SS_X+: now reaches P1.A2 (TX1+)
- net SS_X+: now also P1.B2 (TX2+)
- net SS_X-: now reaches P1.A3 (TX1-)
- net SS_X-: now also P1.B3 (TX2-)
- net DBG_SWC_S: now reaches J1.B2 (TX2+)
- net DBG_SWC_S: now also U8.2 (COM1)
- net DBG_SWD_S: now reaches J1.B3 (TX2-)
- net DBG_SWD_S: now also U8.6 (COM2)
- net DUT_SWC_P: no longer names the net of U4.15 (GPIO12)
- net DUT_SWC_P: no longer U6.2
- net DUT_SWC_P_L renamed DUT_SWC_L
- net DUT_SWC_L: now also U14.11 (S4B), TP1.1; no longer U11.3 (S2B)
- net DUT_SWDIR_P: no longer names the net of U4.14 (GPIO11)
- net DUT_SWDIR_P: no longer U3.5 (DIR)
- net DUT_SWD_P: no longer names the net of U4.16 (GPIO13)
- net DUT_SWD_P: no longer U3.4 (B)
- net DUT_SWD_P_L renamed DUT_SWD_L
- net DUT_SWD_L: now also U14.7 (S3B), TP2.1; no longer U11.15 (S1B)
- net JLK_D+: no longer names the net of U1.8 (DP1+)
- net JLK_D-: no longer names the net of U1.7 (DM1-)
- net USE_PICO renamed DUT_SBU_SWD_ALT
- net DUT_SBU_SWD_ALT: now also R10.2, U7.4
- new net: C2.1, R5.1, U7.3 (+)
- new net: R12.1, R16.2
- new net: R11.2, R12.2, U13.2 (-), U13.6 (-)
- new net: R6.2, R7.2, U7.1 (-)
- new net: R13.2, U13.1, U13.7, U8.3 (IN2), U8.7 (IN1)
Other:
- note added: "SWC"
- note added: "SWD"
- note removed: "JLink"
- moved on the sheet: C1, C14, FB1, R1, R2, R22, R23, SW1, U1, U9, Y1

Commit message: backup
Parts:
- removed C2, C5: 1uF, Capacitor_SMD:C_0603_1608Metric, symbol Device:C_Small
- removed C7: 0.1uF, Capacitor_SMD:C_0603_1608Metric, symbol Device:C_Small
- removed J1: USB_C_Receptacle, Connector_USB:USB_C_Receptacle_Molex_105450-0101, symbol Connector:USB_C_Receptacle
- removed J3: Conn_01x08_Pin, Connector_PinHeader_2.54mm:PinHeader_1x08_P2.54mm_Vertical, symbol Connector:Conn_01x08_Pin
- removed R10, R12, R13, R16, R5, R6, R7: 56k, Resistor_SMD:R_0603_1608Metric, symbol Device:R
- removed R11, R22, R23: 5.1k, Resistor_SMD:R_0603_1608Metric, symbol Device:R
- removed U1: ~, Package_SO:QSOP-16_3.9x4.9mm_P0.635mm, symbol Interface_USB:CH334R
- removed U13: LM2903, Package_DFN_QFN:DFN-8-1EP_2x2mm_P0.5mm_EP0.9x1.6mm, symbol uswc:LM2903DSG
- removed U7: LM397, Package_TO_SOT_SMD:SOT-23-5, symbol Comparator:LM397
- removed U8: TS5A23166DCU, Package_SO:VSSOP-8_2.3x2mm_P0.5mm, symbol uswc:TS5A23166DCU
- removed Y1: 12MHz 10ppm, Crystal:Crystal_SMD_3225-4Pin_3.2x2.5mm, symbol Device:Crystal_GND24
- added J1: USB_C_Receptacle_USB2.0_16P, Connector_USB:USB_C_Receptacle_HRO_TYPE-C-31-M-12, symbol Connector:USB_C_Receptacle_USB2.0_16P
- added U7: CH334F, Package_DFN_QFN:QFN-24-1EP_4x4mm_P0.5mm_EP2.7x2.7mm, symbol ic:CH334F
Connections:
- net +3V3: now also SW1.3 (C), U3.1 (VCCA); no longer U3.6 (VCCB)
- net CC1: now also J1.A5 (CC1)
- net CC2: now also J1.B5 (CC2)
- net D+: now also J1.A6 (D+), J1.B6 (D+), U7.15 (DPU+)
- net D-: now also J1.A7 (D-), J1.B7 (D-), U7.14 (DMU-)
- net DAP_D+: now also U7.12 (DP1+)
- net DAP_D-: now also U7.11 (DM1-)
- net DBG_SWC: now also J1.B8 (SBU2)
- net DBG_SWD: now also J1.A8 (SBU1)
- net DUT_D+: now also U7.6 (DP4+)
- net DUT_D-: now also U7.5 (DM4-)
- net DUT_SBU_SWD_ALT: now also U4.34 (GPIO22)
- net DUT_SWC/D_SBU: now also U4.41 (GPIO29_ADC3)
- net DUT_SWD: now also U3.3 (A); no longer U3.4 (B)
- net DUT_SWD_L: now also U3.4 (B); no longer U3.3 (A)
- net DUT_SWD/C_SBU: now also U4.40 (GPIO28_ADC2)
- net DUT_VREF: now also U3.6 (VCCB); no longer U3.1 (VCCA)
- net GND: now also SW1.1 (A), J1.A1 (GND), J1.A12 (GND), J1.B1 (GND), J1.B12 (GND), U7.25 (GND), U7.4 (XI)
- net SHIELD: now also J1.S1 (SHIELD)
- net VBUS: now also J1.A4 (VBUS), J1.A9 (VBUS), J1.B4 (VBUS), J1.B9 (VBUS), U7.19 (V5)
- net at C1.2: now also U7.20 (VDD33)
- net DFP_CC1: now reaches P1.A5 (CC), R8.1
- net DFP_CC1: now also U4.38 (GPIO26_ADC0)
- net DFP_CC2: now reaches U4.39 (GPIO27_ADC1)
- net DFP_CC2: now also P1.B5 (VCONN), R9.1
- new net: U7.17 (NC), U7.2 (NC)
Other:
- moved on the sheet: C1, C15, R8, R9

Commit message: pend
Parts:
- removed SW1: SW_SPDT, Button_Switch_SMD:SW_SPDT_PCM12, symbol Switch:SW_SPDT
- removed U11, U14: ~, Package_DFN_QFN:UQFN-16_1.8x2.6mm_P0.4mm, symbol misc:FSA2567UMX
- added C2: 1u, Capacitor_SMD:C_0603_1608Metric, symbol Device:C
- added R5, R6: 56k, Resistor_SMD:R_0603_1608Metric, symbol Device:R
- added R7: 5.1k, Resistor_SMD:R_0603_1608Metric, symbol Device:R
- added U1, U8: ADG884xRM, Package_SO:MSOP-10_3x3mm_P0.5mm, symbol Analog_Switch:ADG884xRM
- P1: footprint lib:jingtuojin_918-118A2021Y40005 -> lib:jingtuojin_918-118A2021Y40005-no-ss
Connections:
- net +3V3: now also U1.1 (VDD), U8.1 (VDD)
- net DFP_CC2: now also U4.40 (GPIO28_ADC2); no longer U4.39 (GPIO27_ADC1)
- net DUT_SBU_A: now also U4.41 (GPIO29_ADC3), U1.9 (D2)
- net DUT_SBU_B: now also U4.39 (GPIO27_ADC1), U1.3 (D1)
- net DUT_SWC_L: now also U8.2 (S1A), U8.7 (S2B)
- net DUT_SWC/D_SBU: now also U1.2 (S1A), U8.9 (D2); no longer U4.41 (GPIO29_ADC3)
- net DUT_SWD_L: now also U8.10 (S2A), U8.5 (S1B)
- net DUT_SWD/C_SBU: now also U1.10 (S2A), U8.3 (D1); no longer U4.40 (GPIO28_ADC2)
- net DUT_VREF: now also C2.1, R7.1
- net GND: now also C2.2, R5.1, R6.1, U1.6 (GND), U8.6 (GND)
- net DUT_SWD_CONN: now reaches U4.30 (GPIO19)
- net DUT_SWD_CONN: now also R5.2, U1.4 (IN1), U1.8 (IN2)
- net DUT_SWD_SWAP: now reaches U4.31 (GPIO20)
- net DUT_SWD_SWAP: now also R6.2, U8.4 (IN1), U8.8 (IN2)
- net PWM: now reaches U4.32 (GPIO21)
- net PWM: now also R7.2
- net DUT_SBU_SWD_ALT: no longer names the net of U4.34 (GPIO22)
- removed net SS_X+: P1.A11 (RX2+), P1.A2 (TX1+), P1.B11 (RX1+), P1.B2 (TX2+)
- removed net SS_X-: P1.A10 (RX2-), P1.A3 (TX1-), P1.B10 (RX1-), P1.B3 (TX2-)
- no-connect marks 10 -> 20
Other:
- note removed: "SBU"
- note removed: "SWC"
- note removed: "SWD"
